File: HW/CAD/Eagle/UFBmod_1V0.sch (EAGLE design)
At the start: 27 parts, among them Q0921 ABS07-32.768KHZ, U0611 MR44V064BMAZAATL, U0911 BNO085, U1311 TPS62745DSSR

Commit message: HW_1V0 - CAD/Eagle - Digilent Cmod A7 included, some unwanted sheets removed
Parts:
- removed C0601, C0901, C0903: 100nF, df4iah_rcl:C-EUC0402
- removed C0921, C0922: 22pF, df4iah_rcl:C-EUC0402
- removed Q0921: ABS07-32.768KHZ, df4iah_crystal:ABS07-32.768KHZ
- removed R0511, R0512: 1kR, df4iah_rcl:R-EU_R0402
- removed R0551, R0552: 3R, df4iah_rcl:R-EU_R0402
- removed R0901, R0902, R0904: 33R, df4iah_rcl:R-EU_R0402
- removed R0903: 47R, df4iah_rcl:R-EU_R0402
- removed R0931, R0932: 3.9kR, df4iah_rcl:R-EU_R0402
- removed U0611: MR44V064BMAZAATL, df4iah_memory:FEDR44V064B-02_FRAM_8K-8_I2C
- removed U0911: BNO085, df4iah_sensors:BNO085
- added C101: 100nF, df4iah_rcl:C-EUC0402
- added L101, L102: 300R, df4iah_rcl:R-EU_R1206
- added R111, R112, R113, R114, R121, R131, R141: 47R, df4iah_rcl:R-EU_R0402
- added U101: DIGILENT_CMOD_A7, df4iah_fpga:DIGILENT_CMOD_A7
Connections:
- removed net BNO_CAP: C0903.1, U0911.CAP
- removed net BNO_CLKSEL1_XOUT32: C0922.1, Q0921.1, U0911.CLKSEL1/XOUT32
- removed net BNO_ENV_SCL: R0932.1, U0911.ENV_SCL
- removed net BNO_ENV_SDA: R0931.1, U0911.ENV_SDA
- removed net BNO_H_CSN: R0904.2, U0911.H_CSN
- removed net BNO_INTN: R0902.2, U0911.H_INTN
- removed net BNO_MISO: R0901.2, U0911.H_SDA/MISO/TX
- removed net BNO_PS0_WAKE: R0903.2, U0911.PS0/WAKE
- removed net BNO_XIN32: C0921.1, Q0921.2, U0911.XIN32
- removed net PA10: R0511.1, U0611.SDA
- removed net PA9: R0512.1, U0611.SCL
- removed net PC10: R0552.1
- removed net PC12: R0551.1
- removed net SPI3_MOSI: R0551.2
- removed net SPI3_SCK: R0552.2
- new net +5V: L101.1
- new net FPGA_MISO: R114.1, U101.42_9N
- new net FPGA_MOSI: R113.1, U101.43_13N
- new net FPGA_SCLK: R111.1, U101.45_19P
- new net FPGA_SELN: R112.1, U101.44_9P
- new net FPGA_TRX_CLKO: R141.2, U101.21_10N
- new net FPGA_TRX_IRQ: R121.1, U101.40_12N
- new net FPGA_TRX_RESETN: R131.2, U101.20_9P
- new net TRX_CLKO: R141.1
- new net TRX_IRQ: R121.2
- new net TRX_MISO: R114.2
- new net TRX_MOSI: R113.2
- new net TRX_RESETN: R131.1
- new net TRX_RXCLKN: U101.48_14N
- new net TRX_RXCLKP: U101.47_14P
- new net TRX_RXDN09N: U101.37_11N
- new net TRX_RXDN24N: U101.01_8N
- new net TRX_RXDP09P: U101.38_11P
- new net TRX_RXDP24P: U101.02_8P
- new net TRX_SCLK: R111.2
- new net TRX_SELN: R112.2
- new net TRX_TXCLKN: U101.19_12N
- new net TRX_TXCLKP: U101.18_12P
- new net TRX_TXDN: U101.34_6N
- new net TRX_TXDP: U101.35_6P
- new net VCCA: C101.2, L101.2, U101.24_VU
- new net VSSA: C101.1, L102.2, U101.25_GND
- net +3V3: no longer C0601.2, C0901.1, R0511.2, R0512.2, R0931.2, R0932.2, U0611.VCC, U0911.PS1, U0911.VDD, U0911.VDDIO
- net GND: now also L102.1; no longer C0601.1, C0901.2, C0903.2, C0921.2, C0922.2, U0611.A0, U0611.A1, U0611.A2, U0611.VSS, U0611.WP, U0911.CLKSEL0, U0911.VSS, U0911.VSSIO
Other:
- note added: "Digilent Cmod A7-35T CPG236-1"
- note added: "Microchip AT86RF215"
- note added: "SPI: TRX"
- note removed: "9-axis sensor: BNO-085 SPI"
- note removed: "Addr Device 0x50 FRAM 0x76/0x77 BME280"
- note removed: "Digilent Artix-A7-35"
- note removed: "I2C1 Address space"
- note removed: "I2C1 FRAM 8k x 8b I2C addr: 0x50"
- note removed: "I2C1 Termination"
- note removed: "I2C1: FRAM 64kB"
- note removed: "I2C1_FRAM_SCL"
- note removed: "I2C1_FRAM_SDA"
- note removed: "Iq=130uA"
- note removed: "MCU_I2C1_SCL"
- note removed: "MCU_I2C1_SDA"
- note removed: "Position tracking"
- note removed: "SPI3 MCU --> bus devices"

Commit message: HW_1V0 - CAD/Eagle - schematics for the RF area expanded
Parts:
- removed R141: 47R, df4iah_rcl:R-EU_R0402
- added C311, C312, C406, C407, C408, C511, C551, C552, C553: 100nF, df4iah_rcl:C-EUC0402
- added C321, C401: 1uF, df4iah_rcl:C-EUC0402
- added C403, C404, C521, C531, C532: 1nF, df4iah_rcl:C-EUC0402
- added C411, C412: 10nF, df4iah_rcl:C-EUC0402
- added C413: 56pF, df4iah_rcl:C-EUC0402
- added L401, L402, L403, L404: 300R, df4iah_rcl:R-EU_R1206
- added L421: MURATA DXW21HN5011BL, df4iah_balun:DXW21HN5011BL
- added L422: Johanson 2450BL15B050E, df4iah_balun:2450BL15B050
- added L521: ? nH, df4iah_rcl:L-EUL1812
- added R211, R212: 3.9kR, df4iah_rcl:R-EU_R0402
- added R321: 100kR, df4iah_rcl:R-EU_R0402
- added R413: 100R, df4iah_rcl:R-EU_R0402
- added U301: MAX5217, df4iah_dac:MAX5217
- added U401: AT86RF215-ZU, df4iah_rf:AT86RF215
- added U411: ASVTX-13-D-26.000MHZ-I05-T, df4iah_osc:ASVTX-13-D
- added U511: PE4259, df4iah_rf:PE4259
- added U521: (no value), df4iah_rf:RFX1010
Connections:
- net FPGA_TRX_RESETN renamed FPGA_TRX_RSTN
- removed net TRX_RESETN: R131.1
- removed net TRX_RXDN09N: U101.37_11N
- removed net TRX_RXDN24N: U101.01_8N
- removed net TRX_RXDP09P: U101.38_11P
- removed net TRX_RXDP24P: U101.02_8P
- new net 26MHZ_DAC_OUT: R321.1, U301.OUT
- new net FE09_ANT: L521.2, U521.ANT
- new net FE09_DET: U521.DET
- new net FE09_IND: L521.1, U521.IND
- new net FE09_MODE: U101.23_19N, U521.MODE
- new net FE09_RX: C532.1, U521.RX
- new net FE09_TX: C531.1, U521.TX
- new net FPGA_FE09_DET: U101.15_AD4
- new net FPGA_I2C_SCL: R212.1, U101.26_2P, U301.SCL
- new net FPGA_I2C_SDA: R211.1, U101.27_2N, U301.SDA
- new net PE09_RF1: C531.2, U511.RF1
- new net PE09_RF2: C532.2, U511.RF2
- new net PE09_RFC: C521.1, U511.RFC
- new net TRX_AVDD0: C407.2, U401.AVDD0
- new net TRX_AVDD1: C408.2, U401.AVDD1
- new net TRX_AVSS: C404.2, C407.1, C408.1, L401.2, U401.AVSS
- new net TRX_DEVDD: C403.1, L403.2, U401.DEVDD
- new net TRX_DVDD: C406.2, U401.DVDD
- new net TRX_DVSS: C403.2, C406.1, L402.2, U401.DVSS
- new net TRX_EVDD: C404.1, L404.2, U401.EVDD
- new net TRX_FEA09: U401.FEA09, U511.CTRL, U521.TXEN
- new net TRX_FEA24: U401.FEA24
- new net TRX_FEB09: U401.FEB09, U521.RXEN
- new net TRX_FEB24: U401.FEB24
- new net TRX_RF09: C521.2, L421.UB
- new net TRX_RF09N: L421.B2, U401.RF09N
- new net TRX_RF09P: L421.B1, U401.RF09P
- new net TRX_RF24: L422.UB
- new net TRX_RF24N: L422.B2, U401.RF24N
- new net TRX_RF24P: L422.B1, U401.RF24P
- new net TRX_RSTN: R131.1, U401.RSTN
- new net TRX_RXD09N: U101.37_11N, U401.RXD09N
- new net TRX_RXD09P: U101.38_11P, U401.RXD09P
- new net TRX_RXD24N: U101.01_8N, U401.RXD24N
- new net TRX_RXD24P: U101.02_8P, U401.RXD24P
- new net TRX_TCXO: C412.2, U401.TCXO
- new net VCTCXO_OUT: C412.1, U411.OUT
- new net VCTCXO_VC: C321.1, R321.2, U411.VC
- net +3V3: now also C311.1, C312.1, C401.1, C411.1, C511.1, C551.1, C552.1, C553.1, L403.1, L404.1, R211.2, R212.2, U301.!AUX, U301.REF, U301.VDD, U411.VCC_3V3, U511.VDD_!CTRL, U521.VDD1, U521.VDD2, U521.VDD3
- net FPGA_TRX_CLKO: now also C413.1, R413.1; no longer R141.2
- net GND: now also C311.2, C312.2, C321.2, C401.2, C411.2, C413.2, C511.2, C551.2, C552.2, C553.2, L401.1, L402.1, L421.COM, L422.COM, L422.G_N_D, U301.ADDR, U301.GND, U401.XTAL2, U411.GND, U511.GND, U521.VSS@17, U521.VSS@4, U521.VSS@8
- net TRX_CLKO: now also R413.2, U401.CLKO; no longer R141.1
- net TRX_IRQ: now also U401.IRQ
- net TRX_MISO: now also U401.MISO
- net TRX_MOSI: now also U401.MOSI
- net TRX_RXCLKN: now also U401.RXCLKN
- net TRX_RXCLKP: now also U401.RXCLKP
- net TRX_SCLK: now also U401.SCLK
- net TRX_SELN: now also U401.SELN
- net TRX_TXCLKN: now also U401.TXCLKN
- net TRX_TXCLKP: now also U401.TXCLKP
- net TRX_TXDN: now also U401.TXDN
- net TRX_TXDP: now also U401.TXDP
Other:
- note added: "26MHz"
- note added: "Addr Device 0x38 DAC"
- note added: "Config2 0: OFF 1: ON"
- note added: "Config2 0: RX 1: TX"
- note added: "DAC for VCTCXO pull voltage I2C addr: 0x38"
- note added: "Front end 868 MHz"
- note added: "Front end: LNA & PA for 868 MHz"
- note added: "I2C1 Address space"
- note added: "I2C1 Termination"
- note added: "I2C: DAC"
- note added: "I2C: Termination"
- note added: "Iq=80uA"
- note added: "Microchip Technologies AT86RF215"
- note added: "PMIC 5V --> 3.3V"
- note added: "PMIC: 5V --> 3V3"
- note added: "SAW-Filter: QUALCOMM B3440"
- note added: "TODO"
- note added: "f_LP = 10 Hz"
- note removed: "Microchip AT86RF215"
- note removed: "PMIC --> 3V3"
- note removed: "PMIC 3.3V .. 10V --> 3.3V"

Commit message: HW_1V0 - CAD/Eagle - schematics for the RF area expanded again
Parts:
- removed U1311: TPS62745DSSR, df4iah_powersupply:TPS62745
- removed X2251: (no value), df4iah_connector:HEADER-2X5_1MM27
- added C591, C593: 0pF, df4iah_rcl:C-EUC0402
- added C711: 1nF, df4iah_rcl:C-EUC0402
- added J711: (no value), df4iah_connector:USB_MICRO-B_MOLEX
- added L592: 0nH, df4iah_rcl:L-EUL0603
- added PF711: 1.1A/2.2A, rcl:R-EU_M1206
- added R711: 330kR, df4iah_rcl:R-EU_R0402
- added U581: B39871B3440U410, df4iah_rf:B3440
- added U611: TPS62056DGSR, df4iah_powersupply:TPS62051
- added X599: ANTENNATINY, _c2h:ANTENNATINY
- added X721: (no value), df4iah_connector:HEADER-2X5_1MM27
- C1321: value 10uF -> 22uF
- L1311: value 4.7uH -> 10uH; device df4iah_rcl:L-EUL2520 -> df4iah_rcl:L-EUL1812
- L521: device df4iah_rcl:L-EUL1812 -> df4iah_rcl:L-EUL0603
Connections:
- removed net VBAT_L: C1301.1, U1311.EN, U1311.VIN, U1311.VSEL1, U1311.VSEL2, U1311.VSEL3, U1311.VSEL4
- new net ANT: C593.1, L592.2, X599.SIGNAL
- new net ANT_MATCH: C591.1, L592.1, U581.OUT
- new net USB_SHIELD: C711.2, J711.SHIELD, R711.2
- new net USB_VBUS: J711.J_VUSB, PF711.2
- net +3V3: now also U611.FB; no longer U1311.VOUT
- net +5V: now also C1301.1, PF711.1, U611.EN, U611.VIN
- net FE09_ANT: now also U581.IN
- net GND: now also C591.2, C593.2, C711.1, J711.GND, R711.1, U581.GROUND, U611.LBI, U611.LBO, U611.PG, U611.PGND, U611.SYNC, U611.VSS, X599.GND@0, X599.GND@1, X599.GND@2, X599.GND@3; no longer U1311.EN_VIN_SW, U1311.VSS
- net PMIC3V3_SW: now also U611.SW; no longer U1311.SW
Other:
- note added: "800 mA max."
- note added: "LITTLEFUSE 1206L050YR"
- note added: "MURATA LQH43PN100M26L 4.5mm x 3.2mm (1812)"
- note added: "x599"
- note removed: "300 mA max."
- note removed: "MURATA DFE252010P-4R7M=P2"
- note removed: "SAW-Filter: QUALCOMM B3440"

Commit message: HW_1V0 - CAD/Eagle - board first placement done
Parts:
- renumbered C1301 to C601, C1321 to C621, L1311 to L611
Changed lines of the file:
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@@
 <part name="H2321" library="df4iah_holes" deviceset="MOUNT-PAD-ROUND" device="2.8" value="MOUNT-PAD-ROUND2.8"/>
 <part name="GND2321" library="df4iah_supply" deviceset="GND" device=""/>
-<part name="L1311" library="df4iah_rcl" deviceset="L-EU" device="L1812" value="10uH"/>
-<part name="GND1302" library="df4iah_supply" deviceset="GND" device=""/>
-<part name="C1321" library="df4iah_rcl" deviceset="C-EU" device="C0603" value="22uF"/>
-<part name="GND1301" library="df4iah_supply" deviceset="GND" device=""/>
-<part name="C1301" library="df4iah_rcl" deviceset="C-EU" device="C0603" value="10uF"/>
+<part name="L611" library="df4iah_rcl" deviceset="L-EU" device="L1812" value="10uH"/>
+<part name="GND602" library="df4iah_supply" deviceset="GND" device=""/>
+<part name="C621" library="df4iah_rcl" deviceset="C-EU" device="C0603" value="22uF"/>
+<part name="GND601" library="df4iah_supply" deviceset="GND" device=""/>
+<part name="C601" library="df4iah_rcl" deviceset="C-EU" device="C0603" value="10uF"/>
 <part name="FRAME_22" library="df4iah_frame" deviceset="A4L-LOC" device="" value="Holes"/>
 <part name="X721" library="df4iah_connector" deviceset="HEADER-2X5_1MM27" device="">
@@
 <pinref part="+3V3_301" gate="G$1" pin="+3V3"/>
 <wire x1="86.36" y1="114.3" x2="86.36" y2="109.22" width="0.1524" layer="91"/>
-<pinref part="C311" gate="G$1" pin="1"/>
-<wire x1="129.54" y1="91.44" x2="129.54" y2="88.9" width="0.1524" layer="91"/>
-<pinref part="U301" gate="G$1" pin="REF"/>
-<wire x1="129.54" y1="91.44" x2="119.38" y2="91.44" width="0.1524" layer="91"/>
-<wire x1="86.36" y1="109.22" x2="142.24" y2="109.22" width="0.1524" layer="91"/>
-<wire x1="142.24" y1="109.22" x2="142.24" y2="96.52" width="0.1524" layer="91"/>
+<wire x1="86.36" y1="109.22" x2="147.32" y2="109.22" width="0.1524" layer="91"/>
+<wire x1="147.32" y1="109.22" x2="147.32" y2="96.52" width="0.1524" layer="91"/>
+<wire x1="147.32" y1="96.52" x2="142.24" y2="96.52" width="0.1524" layer="91"/>
+<pinref part="U301" gate="G$1" pin="VDD"/>
 <wire x1="142.24" y1="96.52" x2="119.38" y2="96.52" width="0.1524" layer="91"/>
-<wire x1="142.24" y1="96.52" x2="142.24" y2="91.44" width="0.1524" layer="91"/>
-<junction x="142.24" y="96.52"/>
-<pinref part="U301" gate="G$1" pin="VDD"/>
-<pinref part="C312" gate="G$1" pin="1"/>
-<wire x1="142.24" y1="91.44" x2="142.24" y2="88.9" width="0.1524" layer="91"/>
 <wire x1="86.36" y1="96.52" x2="88.9" y2="96.52" width="0.1524" layer="91"/>
 <wire x1="86.36" y1="96.52" x2="86.36" y2="109.22" width="0.1524" layer="91"/>
 <pinref part="U301" gate="G$1" pin="!AUX"/>
-<wire x1="129.54" y1="91.44" x2="142.24" y2="91.44" width="0.1524" layer="91"/>
+<junction x="86.36" y="109.22"/>
+<pinref part="C312" gate="G$1" pin="1"/>
+<wire x1="142.24" y1="96.52" x2="142.24" y2="88.9" width="0.1524" layer="91"/>
+<junction x="142.24" y="96.52"/>
+<pinref part="U301" gate="G$1" pin="REF"/>
+<pinref part="C311" gate="G$1" pin="1"/>
+<wire x1="129.54" y1="91.44" x2="129.54" y2="88.9" width="0.1524" layer="91"/>
+<wire x1="129.54" y1="91.44" x2="119.38" y2="91.44" width="0.1524" layer="91"/>
+<wire x1="129.54" y1="91.44" x2="147.32" y2="91.44" width="0.1524" layer="91"/>
 <junction x="129.54" y="91.44"/>
-<junction x="142.24" y="91.44"/>
-<junction x="86.36" y="109.22"/>
+<wire x1="147.32" y1="91.44" x2="147.32" y2="96.52" width="0.1524" layer="91"/>
+<junction x="147.32" y="96.52"/>
 </segment>
 </net>
@@
 <attribute name="SHEET" x="230.505" y="5.08" size="2.54" layer="94" font="vector"/>
 </instance>
-<instance part="L1311" gate="G$1" x="160.02" y="116.84" smashed="yes" rot="R270">
+<instance part="L611" gate="G$1" x="160.02" y="116.84" smashed="yes" rot="R270">
 <attribute name="NAME" x="156.21" y="118.3386" size="1.778" layer="95"/>
 <attribute name="VALUE" x="156.21" y="113.538" size="1.778" layer="96"/>
 </instance>
-<instance part="GND1302" gate="1" x="182.88" y="76.2" smashed="yes">
+<instance part="GND602" gate="1" x="182.88" y="76.2" smashed="yes">
 <attribute name="VALUE" x="180.34" y="73.66" size="1.778" layer="96"/>
 </instance>
-<instance part="C1321" gate="G$1" x="182.88" y="101.6" smashed="yes">
+<instance part="C621" gate="G$1" x="182.88" y="101.6" smashed="yes">
 <attribute name="NAME" x="184.404" y="101.981" size="1.778" layer="95"/>
 <attribute name="VALUE" x="184.404" y="96.901" size="1.778" layer="96"/>
 </instance>
-<instance part="GND1301" gate="1" x="81.28" y="76.2" smashed="yes">
+<instance part="GND601" gate="1" x="81.28" y="76.2" smashed="yes">
 <attribute name="VALUE" x="78.74" y="73.66" size="1.778" layer="96"/>
 </instance>
-<instance part="C1301" gate="G$1" x="81.28" y="101.6" smashed="yes">
+<instance part="C601" gate="G$1" x="81.28" y="101.6" smashed="yes">
 <attribute name="NAME" x="82.804" y="101.981" size="1.778" layer="95"/>
 <attribute name="VALUE" x="82.804" y="96.901" size="1.778" layer="96"/>
@@
 <net name="PMIC3V3_SW" class="0">
 <segment>
-<pinref part="L1311" gate="G$1" pin="2"/>
+<pinref part="L611" gate="G$1" pin="2"/>
 <wire x1="147.32" y1="116.84" x2="154.94" y2="116.84" width="0.1524" layer="91"/>
 <pinref part="U611" gate="G$1" pin="SW"/>
@@
 <wire x1="147.32" y1="111.76" x2="172.72" y2="111.76" width="0.1524" layer="91"/>
 <wire x1="172.72" y1="111.76" x2="172.72" y2="116.84" width="0.1524" layer="91"/>
-<pinref part="L1311" gate="G$1" pin="1"/>
+<pinref part="L611" gate="G$1" pin="1"/>
 <wire x1="172.72" y1="116.84" x2="165.1" y2="116.84" width="0.1524" layer="91"/>
 <junction x="172.72" y="116.84"/>
 <wire x1="172.72" y1="116.84" x2="182.88" y2="116.84" width="0.1524" layer="91"/>
 <wire x1="182.88" y1="116.84" x2="200.66" y2="116.84" width="0.1524" layer="91"/>
-<pinref part="C1321" gate="G$1" pin="1"/>
+<pinref part="C621" gate="G$1" pin="1"/>
 <wire x1="182.88" y1="116.84" x2="182.88" y2="104.14" width="0.1524" layer="91"/>
 <junction x="182.88" y="116.84"/>
@@
 <net name="GND" class="0">
 <segment>
-<pinref part="GND1302" gate="1" pin="GND"/>
-<pinref part="C1321" gate="G$1" pin="2"/>
+<pinref part="GND602" gate="1" pin="GND"/>
+<pinref part="C621" gate="G$1" pin="2"/>
 <wire x1="182.88" y1="96.52" x2="182.88" y2="81.28" width="0.1524" layer="91"/>
 <wire x1="182.88" y1="81.28" x2="149.86" y2="81.28" width="0.1524" layer="91"/>
@@
 </segment>
 <segment>
-<pinref part="GND1301" gate="1" pin="GND"/>
-<pinref part="C1301" gate="G$1" pin="2"/>
+<pinref part="GND601" gate="1" pin="GND"/>
+<pinref part="C601" gate="G$1" pin="2"/>
 <wire x1="81.28" y1="78.74" x2="81.28" y2="81.28" width="0.1524" layer="91"/>
 <pinref part="U611" gate="G$1" pin="VSS"/>
@@
 <wire x1="106.68" y1="116.84" x2="104.14" y2="116.84" width="0.1524" layer="91"/>
 <label x="60.96" y="116.84" size="1.778" layer="95" rot="R180" xref="yes"/>
-<pinref part="C1301" gate="G$1" pin="1"/>
+<pinref part="C601" gate="G$1" pin="1"/>
 <wire x1="104.14" y1="116.84" x2="81.28" y2="116.84" width="0.1524" layer="91"/>
 <wire x1="81.28" y1="116.84" x2="60.96" y2="116.84" width="0.1524" layer="91"/>

Commit message: HW_1V0 - CAD/Eagle - routing started, Due to 100R-impedance lines 4layers needed.
Connections:
- net TRX_RF09N renamed TRX_RF09_N
- net TRX_RF09P renamed TRX_RF09_P
- net TRX_RF24N renamed TRX_RF24_N
- net TRX_RF24P renamed TRX_RF24_P
- net TRX_RXCLKN renamed TRX_RXCLK_N
- net TRX_RXCLKP renamed TRX_RXCLK_P
- net TRX_RXD09N renamed TRX_RXD09_N
- net TRX_RXD09P renamed TRX_RXD09_P
- net TRX_RXD24N renamed TRX_RXD24_N
- net TRX_RXD24P renamed TRX_RXD24_P
- net TRX_TXCLKN renamed TRX_TXCLK_N
- net TRX_TXCLKP renamed TRX_TXCLK_P
- net TRX_TXDN renamed TRX_TXD_N
- net TRX_TXDP renamed TRX_TXD_P
- net GND: no longer U401.XTAL2
- net TRX_AVSS: now also U401.XTAL2
Changed lines of the file:
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@@
 <class number="0" name="default" width="0" drill="0.3">
 </class>
-<class number="1" name="pwr_relay" width="1.5" drill="0">
-<clearance class="1" value="0.5"/>
+<class number="1" name="diff_100R" width="0.3" drill="0">
+<clearance class="1" value="0.15"/>
 </class>
 <class number="2" name="pwr_ttl" width="0.75" drill="0">
@@
 <part name="C407" library="df4iah_rcl" deviceset="C-EU" device="C0402" value="100nF"/>
 <part name="C401" library="df4iah_rcl" deviceset="C-EU" device="C0402" value="1uF"/>
-<part name="GND412" library="df4iah_supply" deviceset="GND" device=""/>
 <part name="R413" library="df4iah_rcl" deviceset="R-EU_" device="R0402" value="100R"/>
 <part name="C413" library="df4iah_rcl" deviceset="C-EU" device="C0402" value="56pF"/>
@@
 </busses>
 <nets>
-<net name="TRX_RXD24N" class="0">
+<net name="TRX_RXD24_N" class="1">
 <segment>
 <pinref part="U101" gate="G$1" pin="01_8N"/>
@@
 </segment>
 </net>
-<net name="TRX_RXD24P" class="0">
+<net name="TRX_RXD24_P" class="1">
 <segment>
 <pinref part="U101" gate="G$1" pin="02_8P"/>
@@
 </segment>
 </net>
-<net name="TRX_RXCLKN" class="0">
+<net name="TRX_RXCLK_N" class="1">
 <segment>
 <pinref part="U101" gate="G$1" pin="48_14N"/>
@@
 </segment>
 </net>
-<net name="TRX_RXCLKP" class="0">
+<net name="TRX_RXCLK_P" class="1">
 <segment>
 <pinref part="U101" gate="G$1" pin="47_14P"/>
@@
 </segment>
 </net>
-<net name="TRX_RXD09P" class="0">
+<net name="TRX_RXD09_P" class="1">
 <segment>
 <pinref part="U101" gate="G$1" pin="38_11P"/>
@@
 </segment>
 </net>
-<net name="TRX_RXD09N" class="0">
+<net name="TRX_RXD09_N" class="1">
 <segment>
 <pinref part="U101" gate="G$1" pin="37_11N"/>
@@
 </segment>
 </net>
-<net name="TRX_TXDP" class="0">
+<net name="TRX_TXD_P" class="1">
 <segment>
 <pinref part="U101" gate="G$1" pin="35_6P"/>
@@
 </segment>
 </net>
-<net name="TRX_TXDN" class="0">
+<net name="TRX_TXD_N" class="1">
 <segment>
 <pinref part="U101" gate="G$1" pin="34_6N"/>
@@
 </segment>
 </net>
-<net name="TRX_TXCLKP" class="0">
+<net name="TRX_TXCLK_P" class="1">
 <segment>
 <pinref part="U101" gate="G$1" pin="18_12P"/>
@@
 </segment>
 </net>
-<net name="TRX_TXCLKN" class="0">
+<net name="TRX_TXCLK_N" class="1">
 <segment>
 <pinref part="U101" gate="G$1" pin="19_12N"/>
@@
 </instance>
 <instance part="C401" gate="G$1" x="45.72" y="50.8"/>
-<instance part="GND412" gate="1" x="101.6" y="88.9"/>
 <instance part="R413" gate="G$1" x="86.36" y="83.82"/>
 <instance part="C413" gate="G$1" x="73.66" y="81.28"/>
@@
 <wire x1="86.36" y1="58.42" x2="93.98" y2="58.42" width="0.1524" layer="91"/>
 <junction x="86.36" y="58.42"/>
+<wire x1="86.36" y1="63.5" x2="86.36" y2="76.2" width="0.1524" layer="91"/>
+<junction x="86.36" y="63.5"/>
+<wire x1="86.36" y1="76.2" x2="91.44" y2="76.2" width="0.1524" layer="91"/>
+<wire x1="91.44" y1="76.2" x2="91.44" y2="91.44" width="0.1524" layer="91"/>
+<pinref part="U401" gate="G$1" pin="XTAL2"/>
+<wire x1="91.44" y1="91.44" x2="104.14" y2="91.44" width="0.1524" layer="91"/>
 </segment>
 </net>
@@
 </segment>
 <segment>
-<pinref part="GND412" gate="1" pin="GND"/>
-<pinref part="U401" gate="G$1" pin="XTAL2"/>
-<wire x1="101.6" y1="91.44" x2="104.14" y2="91.44" width="0.1524" layer="91"/>
-</segment>
-<segment>
 <pinref part="C413" gate="G$1" pin="2"/>
 <pinref part="GND413" gate="1" pin="GND"/>
@@
 </segment>
 </net>
-<net name="TRX_RXD24P" class="0">
+<net name="TRX_RXD24_P" class="1">
 <segment>
 <pinref part="U401" gate="G$1" pin="RXD24P"/>
@@
 </segment>
 </net>
-<net name="TRX_RXD24N" class="0">
+<net name="TRX_RXD24_N" class="1">
 <segment>
 <pinref part="U401" gate="G$1" pin="RXD24N"/>
@@
 </segment>
 </net>
-<net name="TRX_RXCLKP" class="0">
+<net name="TRX_RXCLK_P" class="1">
 <segment>
 <pinref part="U401" gate="G$1" pin="RXCLKP"/>
@@
 </segment>
 </net>
-<net name="TRX_RXCLKN" class="0">
+<net name="TRX_RXCLK_N" class="1">
 <segment>
 <pinref part="U401" gate="G$1" pin="RXCLKN"/>
@@
 </segment>
 </net>
-<net name="TRX_RXD09P" class="0">
+<net name="TRX_RXD09_P" class="1">
 <segment>
 <pinref part="U401" gate="G$1" pin="RXD09P"/>
@@
 </segment>
 </net>
-<net name="TRX_RXD09N" class="0">
+<net name="TRX_RXD09_N" class="1">
 <segment>
 <pinref part="U401" gate="G$1" pin="RXD09N"/>
@@
 </segment>
 </net>
-<net name="TRX_TXDP" class="0">
+<net name="TRX_TXD_P" class="1">
 <segment>
 <pinref part="U401" gate="G$1" pin="TXDP"/>
@@
 </segment>
 </net>
-<net name="TRX_TXDN" class="0">
+<net name="TRX_TXD_N" class="1">
 <segment>
 <pinref part="U401" gate="G$1" pin="TXDN"/>
@@
 </segment>
 </net>
-<net name="TRX_TXCLKP" class="0">
+<net name="TRX_TXCLK_P" class="1">
 <segment>
 <pinref part="U401" gate="G$1" pin="TXCLKP"/>
@@
 </segment>
 </net>
-<net name="TRX_TXCLKN" class="0">
+<net name="TRX_TXCLK_N" class="1">
 <segment>
 <pinref part="U401" gate="G$1" pin="TXCLKN"/>
@@
 </segment>
 </net>
-<net name="TRX_RF24N" class="0">
+<net name="TRX_RF24_N" class="0">
 <segment>
 <pinref part="U401" gate="G$1" pin="RF24N"/>
@@
 </segment>
 </net>
-<net name="TRX_RF24P" class="0">
+<net name="TRX_RF24_P" class="0">
 <segment>
 <pinref part="U401" gate="G$1" pin="RF24P"/>
@@
 </segment>
 </net>
-<net name="TRX_RF09P" class="0">
+<net name="TRX_RF09_P" class="1">
 <segment>
 <pinref part="U401" gate="G$1" pin="RF09P"/>
@@
 </segment>
 </net>
-<net name="TRX_RF09N" class="0">
+<net name="TRX_RF09_N" class="1">
 <segment>
 <pinref part="U401" gate="G$1" pin="RF09N"/>
