File: HW/CAD/Eagle/UFBmod_1V0.sch (EAGLE design)
At the start: 63 parts, among them U101 DIGILENT_CMOD_A7, U301 MAX5217, U401 AT86RF215-ZU, U411 ASVTX-13-D-26.000MHZ-I05-T, U511 PE4259, U581 B39871B3440U410, U611 TPS62056DGSR, X599 ANTENNATINY

Commit message: HW_1V0 - CAD/Eagle - connectors added
Parts:
- removed J711: (no value), df4iah_connector:USB_MICRO-B_MOLEX
- added R721, R722, R723, R724: 100R, df4iah_rcl:R-EU_R0402
- added X711: (no value), df4iah_connector:USB_MICRO-B_MOLEX
- added X722, X723: PHOENIX_1990067_1X8X2MM50_PTSA-0-5, df4iah_connector:PHOENIX_1990067_1X8X2MM50_PTSA-0-5
- X721: value (none) -> PHOENIX_1990067_1X8X2MM50_PTSA-0-5; device df4iah_connector:HEADER-2X5_1MM27 -> df4iah_connector:PHOENIX_1990067_1X8X2MM50_PTSA-0-5
Connections:
- new net FPGA_11_16_N: U101.08_11N, X721.8
- new net FPGA_11_16_P: U101.05_11P, X721.7
- new net FPGA_12P16: R721.1, U101.03_12P
- new net FPGA_12P16_R: R721.2, X721.2
- new net FPGA_13P_34: R722.1, U101.46_13P
- new net FPGA_13P_34_R: R722.2, X721.3
- new net FPGA_16_34_N: U101.39_16N, X722.2
- new net FPGA_16_34_P: U101.41_16P, X722.1
- new net FPGA_3P35: R724.1, U101.06_3P
- new net FPGA_3P35_R: R724.2, X721.5
- new net FPGA_3_34_N: U101.29_3P
- new net FPGA_3_34_P: U101.31_3N
- new net FPGA_5_34_N: U101.32_5N, X722.6
- new net FPGA_5_34_P: U101.33_5P, X722.5
- new net FPGA_5_35_N: U101.14_5N, X722.4
- new net FPGA_5_35_P: U101.12_5P, X722.3
- new net FPGA_7N35: R723.1, U101.04_7N
- new net FPGA_7N35_R: R723.2, X721.4
- net GND: now also X711.GND, X721.1, X721.6; no longer J711.GND
- net USB_SHIELD: now also X711.SHIELD; no longer J711.SHIELD
- net USB_VBUS: now also X711.J_VUSB; no longer J711.J_VUSB
Other:
- note added: "X599"
- note removed: "x599"
- moved on the sheet: C711, PF711, R711

Commit message: HW_1V0 - CAD/Eagle - one more line pair added to the connector
Connections:
- net FPGA_3_34_N: now also X722.8
- net FPGA_3_34_P: now also X722.7
Changed lines of the file:
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@@
+</segment>
+</net>
+<net name="FPGA_3_34_P" class="1">
+<segment>
+<pinref part="X722" gate="G$1" pin="7"/>
+<wire x1="228.6" y1="99.06" x2="187.96" y2="99.06" width="0.1524" layer="91"/>
+<label x="187.96" y="99.06" size="1.778" layer="95" rot="R180" xref="yes"/>
+</segment>
+</net>
+<net name="FPGA_3_34_N" class="1">
+<segment>
+<pinref part="X722" gate="G$1" pin="8"/>
+<wire x1="228.6" y1="101.6" x2="137.16" y2="101.6" width="0.1524" layer="91"/>
+<label x="137.16" y="101.6" size="1.778" layer="95" rot="R180" xref="yes"/>
 </segment>
 </net>

Commit message: HW_1V0 - V1.0 at the board house
Parts:
- added C221, C222: 1nF, df4iah_rcl:C-EUC0402
- added C595, C597: 0pF, df4iah_rcl:C-EUC0402
- added D141: ASMT-YTB7-0AA02_RGB, df4iah_led:ASMT-YTB7-0AA02_RGB
- added L596: 0nH, df4iah_rcl:L-EUL0603
- added R141: 180R, df4iah_rcl:R-EU_R0402
- added R142, R143: 130R, df4iah_rcl:R-EU_R0402
- added R151, R152, R521: 1kR, df4iah_rcl:R-EU_R0402
- added R733, R734, R735, R736: 100R, df4iah_rcl:R-EU_R0402
- added X221: TTE_EN11-HSM, df4iah_switch:TTE_EN11-HSM
- added X595: ANTENNATINY, _c2h:ANTENNATINY
- U521: value (none) -> RFX1010
- X711: value (none) -> MOLEX 105017-0001
- renumbered X599 to X591
Connections:
- net ANT renamed ANT09
- net ANT_MATCH renamed ANT09_MATCH
- new net ANT24: C597.1, L596.2, X595.SIGNAL
- new net FPGA_10P35: R736.1, U101.22_10P
- new net FPGA_10P35_R: R736.2, X723.6
- new net FPGA_12P34: R735.1, U101.36_12P
- new net FPGA_12P34_R: R735.2, X723.5
- new net FPGA_1_34_N: U101.30_1N, X723.2
- new net FPGA_1_34_P: U101.28_1P, X723.1
- new net FPGA_9N35: R734.1, U101.17_9N
- new net FPGA_9N35_R: R734.2, X723.4
- new net FPGA_AD12: R733.1, U101.16_AD12
- new net FPGA_AD12_R: R733.2, X723.3
- new net LED_B: D141.BA, R143.1
- new net LED_B_R: R143.2, U101.11_3N
- new net LED_G: D141.GA, R142.1
- new net LED_G_R: R142.2, U101.10_7P
- new net LED_R: D141.RA, R141.1
- new net LED_R_R: R141.2, U101.09_6P
- new net ROT_I: R151.2, U101.07_6N
- new net ROT_I_R: C221.1, R151.1, X221.A
- new net ROT_Q: R152.2, U101.13_6N
- new net ROT_Q_R: C222.1, R152.1, X221.B
- net +3V3: now also X721.6
- net +5V: now also X723.7
- net FE09_DET: now also R521.1
- net FPGA_FE09_DET: now also R521.2
- net GND: now also C221.2, C222.2, C595.2, C597.2, D141.BC, D141.GC, D141.RC, X221.C, X221.D, X595.GND@0, X595.GND@1, X595.GND@2, X595.GND@3, X723.8; no longer U611.LBO, U611.PG, X721.6
- net TRX_RF24: now also C595.1, L596.1
Other:
- note added: "Rotary encoder"
- note added: "X591"
- note added: "X595"
- note removed: "TODO"
- note removed: "X599"
- moved on the sheet: R211, R212
