File: HW/CAD/Eagle/UFBmod_1V0.brd (EAGLE design)
At the start: 78.1 x 89.5 mm, 91 parts, among them U101 DIGILENT_CMOD_A7, U301 MAX5217, U401 AT86RF215-ZU, U411 ASVTX-13-D-26.000MHZ-I05-T, U511 PE4259, U521 RFX1010, U581 B39871B3440U410, U611 TPS62056DGSR, X221 TTE_EN11-HSM, X591 ANTENNATINY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

Commit message: HW_1V0 - CAD/Eagle - LED resistors changed
Parts:
- R141: value 180R -> 820R
- R142: value 130R -> 1kR
- R143: value 130R -> 820R
Changed lines of the file:
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@@
 <attribute name="VALUE" x="58.1025" y="63.1825" size="0.6096" layer="27" font="vector" ratio="10"/>
 </element>
-<element name="R141" library="df4iah_rcl" package="R0402" value="180R" x="55.88" y="34.29" smashed="yes" rot="R180">
+<element name="R141" library="df4iah_rcl" package="R0402" value="820R" x="55.88" y="34.29" smashed="yes" rot="R180">
 <attribute name="NAME" x="54.9275" y="35.08375" size="0.6096" layer="25" font="vector" ratio="10"/>
 <attribute name="VALUE" x="57.4675" y="35.8775" size="0.6096" layer="27" font="vector" ratio="10" rot="R180"/>
 </element>
-<element name="R142" library="df4iah_rcl" package="R0402" value="130R" x="55.88" y="36.83" smashed="yes" rot="R180">
+<element name="R142" library="df4iah_rcl" package="R0402" value="1kR" x="55.88" y="36.83" smashed="yes" rot="R180">
 <attribute name="NAME" x="54.9275" y="37.62375" size="0.6096" layer="25" font="vector" ratio="10"/>
 <attribute name="VALUE" x="57.4675" y="38.4175" size="0.6096" layer="27" font="vector" ratio="10" rot="R180"/>
 </element>
-<element name="R143" library="df4iah_rcl" package="R0402" value="130R" x="55.88" y="39.37" smashed="yes" rot="R180">
+<element name="R143" library="df4iah_rcl" package="R0402" value="820R" x="55.88" y="39.37" smashed="yes" rot="R180">
 <attribute name="NAME" x="54.9275" y="40.16375" size="0.6096" layer="25" font="vector" ratio="10"/>
 <attribute name="VALUE" x="57.4675" y="40.9575" size="0.6096" layer="27" font="vector" ratio="10" rot="R180"/>
