File: HW/CAD/Eagle/UFBmod_2V0.brd (EAGLE design)
At the start: 98.4 x 89.5 mm, 139 parts, among them T0551 MMBT2222, U0501 MIDAS_MCCOG21605B6W-FPTLWI, U0601 MAX5217, U0701 AT86RF215-ZU, U0711 ASVTX-13-D-26.000MHZ-I05-T, U0811 PE4259, U0821 RFX1010, U0881 B39871B3440U410, U1101 TPS53353, U1211 TPS62745DSSR, X0891 ANTENNATINY, X0895 ANTENNATINY, X1011 TTE_EN11-HSM, X1311 MOLEX 105017-0001, X1321 PHOENIX_1990067_1X8X2MM50_PTS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, X1322 PHOENIX_1990067_1X8X2MM50_PTS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, X1323 PHOENIX_1990067_1X8X2MM50_PTS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

Commit message: HW_2V0 - HW/CAD/Eagle - FT232HL added
Parts:
- added C0911, C0912, C0913, C0921, C0922: 100nF, df4iah_rcl:C0402
- added D0971: GREEN, df4iah_led:U57X32
- added D0972: RED, df4iah_led:U57X32
- added L0911, L0921, L0922: 300R, df4iah_rcl:R1206
- added R0911: 12kR 1%0, df4iah_rcl:R0402
- added R0912, R0941, R0961, R0962, R0963, R0964, R0965, R0966, R0967, R0968: 100R, df4iah_rcl:R0402
- added R0913: 100kR, df4iah_rcl:R0402
- added R0931: 10kR, df4iah_rcl:R0402
- added R0971, R0972: 1kR, df4iah_rcl:R0402
- added U0911: FT232HL, df4iah_dataconvertion:LQFP48
- JB1, JB2: value (none) -> LSHM-150-04.0-L-DV-A-S-K-TR
- JB3: value (none) -> LSHM-130-04.0-L-DV-A-S-K-TR
- X1331: device df4iah_connector:2X07_SHROUDED_JTAG_XILINX -> df4iah_connector:2X07_2MM00_SHROUDED_XILINX_JTAG
- moved R1337 3.18 mm to (42.5, 68.6)
- moved R1334 1.27 mm to (48.3, 68.6)
- moved X1331 1.27 mm to (48.3, 73.7)
- moved R1333 0.63 mm to (50.2, 68.6)
Connections:
- new net FPGA_FT_12MHZ: R0941.1
- new net FPGA_FT_CTS: R0964.2
- new net FPGA_FT_DCD: R0967.2
- new net FPGA_FT_DSR: R0966.2
- new net FPGA_FT_DTR: R0965.2
- new net FPGA_FT_RESET: R0912.1
- new net FPGA_FT_RI: R0968.2
- new net FPGA_FT_RTS: R0963.2
- new net FPGA_FT_RXD: R0962.2
- new net FPGA_FT_TXD: R0961.2
- new net FT_AGND: L0911.2, U0911.4, U0911.41, U0911.9
- new net FT_CTS: R0964.1, U0911.16
- new net FT_DCD: R0967.1, U0911.19
- new net FT_DSR: R0966.1, U0911.18
- new net FT_DTR: R0965.1, U0911.17
- new net FT_EEDATA: R0931.1, U0911.43
- new net FT_OSCI: R0941.2, U0911.1
- new net FT_REF: R0911.2, U0911.5
- new net FT_RESET: R0912.2, R0913.2, U0911.34
- new net FT_RI: R0968.1, U0911.20
- new net FT_RTS: R0963.1, U0911.15
- new net FT_RXD: R0962.1, U0911.14
- new net FT_RXLED: R0971.1, U0911.27
- new net FT_RXLED_D: D0971.A, R0971.2
- new net FT_TXD: R0961.1, U0911.13
- new net FT_TXDEN: U0911.21
- new net FT_TXLED: R0972.1, U0911.28
- new net FT_TXLED_D: D0972.A, R0972.2
- new net FT_VCCA: C0913.2, U0911.37
- new net FT_VCCCORE: C0912.2, U0911.38
- new net FT_VCCD: L0921.2, L0922.2, R0931.2, U0911.12, U0911.24, U0911.39, U0911.46
- new net FT_VPHY: C0922.2, L0922.1, U0911.3
- new net FT_VPLL: C0921.2, L0921.1, U0911.8
- net +3V3: now also C0911.1, U0911.40
- net GND: now also C0911.2, C0912.1, C0913.1, C0921.1, C0922.1, D0971.K, D0972.K, L0911.1, R0911.1, R0913.1, U0911.10, U0911.11, U0911.22, U0911.23, U0911.35, U0911.36, U0911.42, U0911.47, U0911.48
- net USB_D_M: now also U0911.6
- net USB_D_P: now also U0911.7
