File: HW/CAD/Eagle/UFBmod_2V0.sch (EAGLE design)
At the start: 135 parts, among them T0551 MMBT2222, U0501 MIDAS_MCCOG21605B6W-FPTLWI, U0601 MAX5217, U0701 AT86RF215-ZU, U0711 ASVTX-13-D-26.000MHZ-I05-T, U0811 PE4259, U0821 RFX1010, U0881 B39871B3440U410, U1101 TPS53353, U1211 TPS62745DSSR, X0891 ANTENNATINY, X0895 ANTENNATINY, X1011 TTE_EN11-HSM, X1311 MOLEX 105017-0001, X1321 PHOENIX_1990067_1X8X2MM50_PTS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, X1322 PHOENIX_1990067_1X8X2MM50_PTS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, X1323 PHOENIX_1990067_1X8X2MM50_PTS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

Commit message: HW_2V0 - HW/CAD/Eagle - FT232HL added
Parts:
- added C0911, C0912, C0913, C0921, C0922: 100nF, df4iah_rcl:C-EUC0402
- added D0971: GREEN, df4iah_led:U57X32
- added D0972: RED, df4iah_led:U57X32
- added L0911, L0921, L0922: 300R, df4iah_rcl:R-EU_R1206
- added R0911: 12kR 1%0, df4iah_rcl:R-EU_R0402
- added R0912, R0941, R0961, R0962, R0963, R0964, R0965, R0966, R0967, R0968: 100R, df4iah_rcl:R-EU_R0402
- added R0913: 100kR, df4iah_rcl:R-EU_R0402
- added R0931: 10kR, df4iah_rcl:R-EU_R0402
- added R0971, R0972: 1kR, df4iah_rcl:R-EU_R0402
- added U0911: FT232HL, df4iah_dataconvertion:FTDI232HL
- JB1, JB2: value (none) -> LSHM-150-04.0-L-DV-A-S-K-TR
- JB3: value (none) -> LSHM-130-04.0-L-DV-A-S-K-TR
Connections:
- new net FPGA_FT_12MHZ: R0941.1
- new net FPGA_FT_CTS: R0964.2
- new net FPGA_FT_DCD: R0967.2
- new net FPGA_FT_DSR: R0966.2
- new net FPGA_FT_DTR: R0965.2
- new net FPGA_FT_RESET: R0912.1
- new net FPGA_FT_RI: R0968.2
- new net FPGA_FT_RTS: R0963.2
- new net FPGA_FT_RXD: R0962.2
- new net FPGA_FT_TXD: R0961.2
- new net FT_AGND: L0911.2, U0911.AGND@4, U0911.AGND@41, U0911.AGND@9
- new net FT_CTS: R0964.1, U0911.ADBUS3
- new net FT_DCD: R0967.1, U0911.ADBUS6
- new net FT_DSR: R0966.1, U0911.ADBUS5
- new net FT_DTR: R0965.1, U0911.ADBUS4
- new net FT_EEDATA: R0931.1, U0911.EEDATA
- new net FT_OSCI: R0941.2, U0911.OSCI
- new net FT_REF: R0911.2, U0911.REF
- new net FT_RESET: R0912.2, R0913.2, U0911.!RESET
- new net FT_RI: R0968.1, U0911.ADBUS7
- new net FT_RTS: R0963.1, U0911.ADBUS2
- new net FT_RXD: R0962.1, U0911.ADBUS1
- new net FT_RXLED: R0971.1, U0911.ACBUS3
- new net FT_RXLED_D: D0971.A, R0971.2
- new net FT_TXD: R0961.1, U0911.ADBUS0
- new net FT_TXDEN: U0911.ACBUS0
- new net FT_TXLED: R0972.1, U0911.ACBUS4
- new net FT_TXLED_D: D0972.A, R0972.2
- new net FT_VCCA: C0913.2, U0911.VCCA
- new net FT_VCCCORE: C0912.2, U0911.VCCCORE
- new net FT_VCCD: L0921.2, L0922.2, R0931.2, U0911.VCCD, U0911.VCCIO@12, U0911.VCCIO@24, U0911.VCCIO@46
- new net FT_VPHY: C0922.2, L0922.1, U0911.VPHY
- new net FT_VPLL: C0921.2, L0921.1, U0911.VPLL
- net +3V3: now also C0911.1, U0911.VREGIN
- net GND: now also C0911.2, C0912.1, C0913.1, C0921.1, C0922.1, D0971.C, D0972.C, L0911.1, R0911.1, R0913.1, U0911.GND@10, U0911.GND@11, U0911.GND@22, U0911.GND@23, U0911.GND@35, U0911.GND@36, U0911.GND@47, U0911.GND@48, U0911.TEST
- net USB_D_M: now also U0911.D_M
- net USB_D_P: now also U0911.D_P
Other:
- note added: "USB / UART FT232H"
- note removed: "FTDI xxxx"
- moved on the sheet: X1331
