File: HW/CAD/Eagle/UFBmod_2V0.sch (EAGLE design)
At the start: 189 parts, among them T0551 MMBT2222, U0501 MIDAS_MCCOG21605B6W-FPTLWI, U0601 MAX5217, U0701 AT86RF215-ZU, U0711 ASVTX-13-D-26.000MHZ-I05-T, U0811 PE4259, U0821 RFX1010, U0881 B39871B3440U410, U0911 FT232HL, U1101 TPS53353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

Commit message: HW - CAD/Eagle - update FPGA assignments
Parts:
- removed C0713: 56pF, df4iah_rcl:C-EUC0402
- removed R0713: 100R, df4iah_rcl:R-EU_R0402
- added TP1371: TPB1,27, df4iah_connector:TPB1,27
- renumbered C1350 to C1381, X1350 to X1381
Connections:
- net FPGA_I2C_SCL renamed BOARD_SCL
- net FPGA_I2C_SDA renamed BOARD_SDA
- net FPGA_LCD_NRST renamed BOARD_LCD_RESETN
- removed net FPGA_TRX_CLKO: C0713.1, JB1.B16_L12_CLK_P, R0713.1
- removed net TRX_CLKO: R0713.2, U0701.CLKO
- new net INIT_CALIB_COMPLETE: TP1371.TP
- net FPGA_LCD_BL_PWM: no longer JB1.B16_L8_P
- net FPGA_LED_RGB_BLUE: no longer JB1.B16_L24_N
- net FPGA_LED_RGB_GREEN: no longer JB1.B16_L22_N
- net FPGA_LED_RGB_RED: no longer JB1.B16_L22_P
- net GND: no longer C0713.2

Commit message: HW - CAD/Eagle - update FPGA assignments
Connections:
- removed net FPGA_ROT_I: R1011.2
- removed net FPGA_ROT_P: R1013.2
- removed net FPGA_ROT_Q: R1012.2
- new net BOARD_ROTENC_I: JB2.B14_L14_CLK_P, R1011.2
- new net BOARD_ROTENC_PUSH: JB2.B14_L13_CLK_P, R1013.2
- new net BOARD_ROTENC_Q: JB2.B14_L14_CLK_N, R1012.2
Other:
- note added: "PULLUP in FPGA to be enabled !"
Changed lines of the file:
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@@
+</segment>
+</net>
+<net name="BOARD_ROTENC_I" class="0">
+<segment>
+<pinref part="JB2" gate="G$1" pin="B14_L14_CLK_P"/>
+<wire x1="96.52" y1="127" x2="40.64" y2="127" width="0.1524" layer="91"/>
+<label x="40.64" y="127" size="1.778" layer="95" rot="R180" xref="yes"/>
+</segment>
+</net>
+<net name="BOARD_ROTENC_Q" class="0">
+<segment>
+<pinref part="JB2" gate="G$1" pin="B14_L14_CLK_N"/>
+<wire x1="96.52" y1="124.46" x2="76.2" y2="124.46" width="0.1524" layer="91"/>
+<label x="76.2" y="124.46" size="1.778" layer="95" rot="R180" xref="yes"/>
+</segment>
+</net>
+<net name="BOARD_ROTENC_PUSH" class="0">
+<segment>
+<pinref part="JB2" gate="G$1" pin="B14_L13_CLK_P"/>
+<wire x1="96.52" y1="121.92" x2="40.64" y2="121.92" width="0.1524" layer="91"/>
+<label x="40.64" y="121.92" size="1.778" layer="95" rot="R180" xref="yes"/>
 </segment>
 </net>
@@
 <text x="182.88" y="162.56" size="2.54" layer="97" ratio="15">RGB LEDs</text>
 <text x="165.1" y="15.24" size="2.54" layer="97" ratio="15">User Control</text>
+<text x="101.6" y="139.7" size="1.778" layer="97">PULLUP in FPGA to be enabled !</text>
 </plain>
 <instances>
@@
 </segment>
 </net>
-<net name="FPGA_ROT_I" class="0">
+<net name="BOARD_ROTENC_I" class="0">
 <segment>
 <pinref part="R1011" gate="G$1" pin="2"/>
@@
 </segment>
 </net>
-<net name="FPGA_ROT_Q" class="0">
+<net name="BOARD_ROTENC_Q" class="0">
 <segment>
 <pinref part="R1012" gate="G$1" pin="2"/>
@@
 </segment>
 </net>
-<net name="FPGA_ROT_P" class="0">
+<net name="BOARD_ROTENC_PUSH" class="0">
 <segment>
 <pinref part="R1013" gate="G$1" pin="2"/>

Commit message: HW_2V0 - CAD/Eagle - RESET button added
Parts:
- added R1321: 100R, df4iah_rcl:R-EU_R0402
- added S1321: KSR223G_SMD_1POL, df4iah_switch:KSR223G_SMD_1POL
Connections:
- new net FPGA_RESET: JB3.B13_L1_N, JB3.B13_L1_P, R1321.1
- new net FPGA_RESET_R: R1321.2, S1321.P
- net VCCIO13: now also S1321.S
Changed lines of the file:
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@@
 <part name="R0754" library="df4iah_rcl" deviceset="R-EU_" device="R0402" value="100R"/>
 <part name="TP1371" library="df4iah_connector" deviceset="TP" device="B1,27"/>
+<part name="S1321" library="df4iah_switch" deviceset="KSR223G_SMD_1POL" device=""/>
+<part name="R1321" library="df4iah_rcl" deviceset="R-EU_" device="R0402" value="100R"/>
 </parts>
 <sheets>
@@
 </segment>
 </net>
+<net name="FPGA_RESET" class="0">
+<segment>
+<pinref part="JB3" gate="G$1" pin="B13_L1_P"/>
+<wire x1="144.78" y1="124.46" x2="144.78" y2="137.16" width="0.1524" layer="91"/>
+<wire x1="144.78" y1="137.16" x2="147.32" y2="137.16" width="0.1524" layer="91"/>
+<pinref part="JB3" gate="G$1" pin="B13_L1_N"/>
+<wire x1="147.32" y1="137.16" x2="147.32" y2="124.46" width="0.1524" layer="91"/>
+<wire x1="144.78" y1="137.16" x2="50.8" y2="137.16" width="0.1524" layer="91"/>
+<junction x="144.78" y="137.16"/>
+<label x="50.8" y="137.16" size="1.778" layer="95" rot="R180" xref="yes"/>
+</segment>
+</net>
 </nets>
 </sheet>
@@
 <instance part="GND1381" gate="1" x="198.12" y="60.96"/>
 <instance part="TP1371" gate="G$1" x="220.98" y="81.28"/>
+<instance part="S1321" gate="G$1" x="114.3" y="53.34"/>
+<instance part="R1321" gate="G$1" x="114.3" y="40.64" rot="R90"/>
 </instances>
 <busses>
@@
 </segment>
 </net>
+<net name="VCCIO13" class="0">
+<segment>
+<pinref part="S1321" gate="G$1" pin="S"/>
+<wire x1="114.3" y1="58.42" x2="114.3" y2="66.04" width="0.1524" layer="91"/>
+<label x="114.3" y="66.04" size="1.778" layer="95" rot="R90" xref="yes"/>
+</segment>
+</net>
+<net name="FPGA_RESET" class="0">
+<segment>
+<pinref part="R1321" gate="G$1" pin="1"/>
+<wire x1="114.3" y1="35.56" x2="114.3" y2="33.02" width="0.1524" layer="91"/>
+<wire x1="114.3" y1="33.02" x2="129.54" y2="33.02" width="0.1524" layer="91"/>
+<label x="129.54" y="33.02" size="1.778" layer="95" xref="yes"/>
+</segment>
+</net>
+<net name="FPGA_RESET_R" class="0">
+<segment>
+<pinref part="R1321" gate="G$1" pin="2"/>
+<pinref part="S1321" gate="G$1" pin="P"/>
+<wire x1="114.3" y1="45.72" x2="114.3" y2="48.26" width="0.1524" layer="91"/>
+</segment>
+</net>

Commit message: HW_2V0 - CAD/Eagle - signal name change
Connections:
- net INIT_CALIB_COMPLETE renamed DDR3_INIT_CALIB_COMPLETE
Changed lines of the file:
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@@
 </segment>
 </net>
-<net name="INIT_CALIB_COMPLETE" class="0">
+<net name="DDR3_INIT_CALIB_COMPLETE" class="0">
 <segment>
 <wire x1="96.52" y1="137.16" x2="76.2" y2="137.16" width="0.1524" layer="91"/>
@@
 </segment>
 </net>
-<net name="INIT_CALIB_COMPLETE" class="0">
+<net name="DDR3_INIT_CALIB_COMPLETE" class="0">
 <segment>
 <wire x1="220.98" y1="76.2" x2="177.8" y2="76.2" width="0.1524" layer="91"/>

Commit message: HW_2V0 - CAD/Eagle - Ethernet Link-LED added
Connections:
- net FPGA_ETH_DA_G: now also JB2.B14_L17_P
- net FPGA_ETH_DA_Y: now also JB2.B14_L17_N
Changed lines of the file:
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@@
+</segment>
+</net>
+<net name="FPGA_ETH_DA_Y" class="0">
+<segment>
+<pinref part="JB2" gate="G$1" pin="B14_L17_N"/>
+<wire x1="96.52" y1="134.62" x2="40.64" y2="134.62" width="0.1524" layer="91"/>
+<label x="40.64" y="134.62" size="1.778" layer="95" rot="R180" xref="yes"/>
+</segment>
+</net>
+<net name="FPGA_ETH_DA_G" class="0">
+<segment>
+<pinref part="JB2" gate="G$1" pin="B14_L17_P"/>
+<wire x1="96.52" y1="132.08" x2="76.2" y2="132.08" width="0.1524" layer="91"/>
+<label x="76.2" y="132.08" size="1.778" layer="95" rot="R180" xref="yes"/>
 </segment>
 </net>

Commit message: HW_2V0 - CAD/Eagle - connect TRX VC-TCXO 26MHz with FPGA
Parts:
- added R0711: 100R, df4iah_rcl:R-EU_R0402
Connections:
- new net TRX_CLKO_26MHZ_R: R0711.2, U0701.CLKO
- new net TRX_CLK_26MHZ: JB2.B15_L11_CLK_P, R0711.1
Changed lines of the file:
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@@
 <part name="S1321" library="df4iah_switch" deviceset="KSR223G_SMD_1POL" device=""/>
 <part name="R1321" library="df4iah_rcl" deviceset="R-EU_" device="R0402" value="100R"/>
+<part name="R0711" library="df4iah_rcl" deviceset="R-EU_" device="R0402" value="100R"/>
 </parts>
 <sheets>
@@
 <wire x1="96.52" y1="132.08" x2="76.2" y2="132.08" width="0.1524" layer="91"/>
 <label x="76.2" y="132.08" size="1.778" layer="95" rot="R180" xref="yes"/>
+</segment>
+</net>
+<net name="TRX_CLK_26MHZ" class="0">
+<segment>
+<pinref part="JB2" gate="G$1" pin="B15_L11_CLK_P"/>
+<wire x1="96.52" y1="88.9" x2="76.2" y2="88.9" width="0.1524" layer="91"/>
+<label x="76.2" y="88.9" size="1.778" layer="95" rot="R180" xref="yes"/>
 </segment>
 </net>
@@
 <instance part="R0753" gate="G$1" x="200.66" y="58.42"/>
 <instance part="R0754" gate="G$1" x="185.42" y="53.34"/>
+<instance part="R0711" gate="G$1" x="73.66" y="83.82"/>
 </instances>
 <busses>
@@
 </segment>
 </net>
+<net name="TRX_CLKO_26MHZ_R" class="0">
+<segment>
+<pinref part="U0701" gate="G$1" pin="CLKO"/>
+<wire x1="104.14" y1="83.82" x2="78.74" y2="83.82" width="0.1524" layer="91"/>
+<pinref part="R0711" gate="G$1" pin="2"/>
+</segment>
+</net>
+<net name="TRX_CLK_26MHZ" class="0">
+<segment>
+<pinref part="R0711" gate="G$1" pin="1"/>
+<wire x1="68.58" y1="83.82" x2="45.72" y2="83.82" width="0.1524" layer="91"/>
+<label x="45.72" y="83.82" size="1.778" layer="95" rot="R180" xref="yes"/>
+</segment>
+</net>
