File: HW/CAD/Eagle/UFBmod_2V1.sch (EAGLE design)
At the start: 193 parts, among them T0551 MMBT2222, U0501 MIDAS_MCCOG21605B6W-FPTLWI, U0601 MAX5217, U0701 AT86RF215-ZU, U0711 ASVTX-13-D-26.000MHZ-I05-T, U0811 PE4259, U0821 RFX1010, U0881 B39871B3440U410, U0911 FT232HL, U1101 TPS53353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

Commit message: HW_2V1 - CAD/Eagle - ERC done
Parts:
- added R0203: 10kR, df4iah_rcl:R-EU_R0402
- added TP_EN1, TP_MODE, TP_PGOOD, TP_RESIN, TP_RFX_DET, TP_TXDEN: TPB1,27, df4iah_connector:TPB1,27
- J1411: value (none) -> ABRACON_ARJE-0034
Connections:
- new net FPGA_EN1: JB1.EN1@27, TP_EN1.TP
- new net FPGA_MODE: JB1.MODE@31, TP_MODE.TP
- new net PGOOD: JB1.PGOOD@29, TP_PGOOD.TP
- new net RESIN: JB2.RESIN, R0203.1, TP_RESIN.TP
- net +3V3: now also R0203.2
- net FPGA_RFX_DET: now also TP_RFX_DET.TP
- net FT_TXDEN: now also TP_TXDEN.TP

Commit message: HW_2V1 - CAD/Eagle - DRC work-of-the-day
Parts:
- renumbered TP_EN1 to FPGA_EN1, TP_MODE to FPGA_MODE, TP_PGOOD to PGOOD
Changed lines of the file:
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@@
 <part name="C0713" library="df4iah_rcl" deviceset="C-EU" device="C0402" value="1nF"/>
 <part name="GND0712" library="df4iah_supply" deviceset="GND" device=""/>
-<part name="TP_EN1" library="df4iah_connector" deviceset="TP" device="B1,27"/>
-<part name="TP_PGOOD" library="df4iah_connector" deviceset="TP" device="B1,27"/>
-<part name="TP_MODE" library="df4iah_connector" deviceset="TP" device="B1,27"/>
+<part name="FPGA_EN1" library="df4iah_connector" deviceset="TP" device="B1,27"/>
+<part name="PGOOD" library="df4iah_connector" deviceset="TP" device="B1,27"/>
+<part name="FPGA_MODE" library="df4iah_connector" deviceset="TP" device="B1,27"/>
 <part name="TP_RESIN" library="df4iah_connector" deviceset="TP" device="B1,27"/>
 <part name="R0203" library="df4iah_rcl" deviceset="R-EU_" device="R0402" value="10kR"/>
@@
 <instance part="JB1" gate="G$1" x="129.54" y="91.44"/>
 <instance part="+3V3_0101" gate="G$1" x="38.1" y="152.4" rot="R90"/>
-<instance part="TP_EN1" gate="G$1" x="182.88" y="119.38" smashed="yes" rot="R270">
+<instance part="FPGA_EN1" gate="G$1" x="182.88" y="119.38" smashed="yes" rot="R270">
 <attribute name="NAME" x="184.15" y="118.11" size="1.778" layer="95"/>
 <attribute name="TP_SIGNAL_NAME" x="181.61" y="118.11" size="1.778" layer="97" rot="R270"/>
 </instance>
-<instance part="TP_PGOOD" gate="G$1" x="203.2" y="116.84" smashed="yes" rot="R270">
+<instance part="PGOOD" gate="G$1" x="203.2" y="116.84" smashed="yes" rot="R270">
 <attribute name="NAME" x="204.47" y="115.57" size="1.778" layer="95"/>
 <attribute name="TP_SIGNAL_NAME" x="201.93" y="115.57" size="1.778" layer="97" rot="R270"/>
 </instance>
-<instance part="TP_MODE" gate="G$1" x="182.88" y="114.3" smashed="yes" rot="R270">
+<instance part="FPGA_MODE" gate="G$1" x="182.88" y="114.3" smashed="yes" rot="R270">
 <attribute name="NAME" x="184.15" y="113.03" size="1.778" layer="95"/>
 <attribute name="TP_SIGNAL_NAME" x="181.61" y="113.03" size="1.778" layer="97" rot="R270"/>
@@
 <pinref part="JB1" gate="G$1" pin="EN1@27"/>
 <wire x1="162.56" y1="119.38" x2="180.34" y2="119.38" width="0.1524" layer="91"/>
-<pinref part="TP_EN1" gate="G$1" pin="TP"/>
+<pinref part="FPGA_EN1" gate="G$1" pin="TP"/>
 </segment>
 </net>
@@
 <pinref part="JB1" gate="G$1" pin="PGOOD@29"/>
 <wire x1="162.56" y1="116.84" x2="200.66" y2="116.84" width="0.1524" layer="91"/>
-<pinref part="TP_PGOOD" gate="G$1" pin="TP"/>
+<pinref part="PGOOD" gate="G$1" pin="TP"/>
 </segment>
 </net>
@@
 <pinref part="JB1" gate="G$1" pin="MODE@31"/>
 <wire x1="162.56" y1="114.3" x2="180.34" y2="114.3" width="0.1524" layer="91"/>
-<pinref part="TP_MODE" gate="G$1" pin="TP"/>
-</segment>
-</net>
+<pinref part="FPGA_MODE" gate="G$1" pin="TP"/>
+</segment>
+</net>

Commit message: HW_2V1 - CAD/Eagle - some minor fixes
Parts:
- removed C593: 0pF, df4iah_rcl:C-EUC0402
- added C0893: 0pF, df4iah_rcl:C-EUC0402
Connections:
- net ANT09: now also C0891.1; no longer C593.1
- net ANT09_MATCH: now also C0893.1; no longer C0891.1
- net ANT24: now also C0895.1; no longer C0897.1
- net GND: now also C0893.2; no longer C593.2
- net TRX_RF24: now also C0897.1; no longer C0895.1
Other:
- moved on the sheet: C0891, C0895, C0897
Changed lines of the file:
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@@
 <part name="GND0852" library="df4iah_supply" deviceset="GND" device=""/>
 <part name="GND0851" library="df4iah_supply" deviceset="GND" device=""/>
-<part name="C593" library="df4iah_rcl" deviceset="C-EU" device="C0402" value="0pF"/>
+<part name="C0891" library="df4iah_rcl" deviceset="C-EU" device="C0402" value="0pF"/>
 <part name="L0892" library="df4iah_rcl" deviceset="L-EU" device="L0603" value="0nH"/>
-<part name="C0891" library="df4iah_rcl" deviceset="C-EU" device="C0402" value="0pF"/>
+<part name="C0893" library="df4iah_rcl" deviceset="C-EU" device="C0402" value="0pF"/>
 <part name="GND0893" library="df4iah_supply" deviceset="GND" device=""/>
 <part name="GND0891" library="df4iah_supply" deviceset="GND" device=""/>
@@
 <part name="X0895" library="_c2h" deviceset="ANTENNA" device="TINY"/>
 <part name="GND0898" library="df4iah_supply" deviceset="GND" device=""/>
+<part name="C0895" library="df4iah_rcl" deviceset="C-EU" device="C0402" value="0pF"/>
 <part name="C0897" library="df4iah_rcl" deviceset="C-EU" device="C0402" value="0pF"/>
-<part name="C0895" library="df4iah_rcl" deviceset="C-EU" device="C0402" value="0pF"/>
 <part name="L0896" library="df4iah_rcl" deviceset="L-EU" device="L0603" value="0nH"/>
 <part name="GND0897" library="df4iah_supply" deviceset="GND" device=""/>
@@
 <instance part="GND0852" gate="1" x="106.68" y="66.04"/>
 <instance part="GND0851" gate="1" x="116.84" y="66.04"/>
-<instance part="C593" gate="G$1" x="20.32" y="109.22"/>
+<instance part="C0891" gate="G$1" x="20.32" y="109.22"/>
 <instance part="L0892" gate="G$1" x="27.94" y="116.84" rot="R270"/>
-<instance part="C0891" gate="G$1" x="35.56" y="109.22"/>
+<instance part="C0893" gate="G$1" x="35.56" y="109.22"/>
 <instance part="GND0893" gate="1" x="20.32" y="99.06"/>
 <instance part="GND0891" gate="1" x="35.56" y="99.06"/>
@@
 <instance part="X0895" gate="1" x="10.16" y="35.56" rot="MR0"/>
 <instance part="GND0898" gate="1" x="12.7" y="17.78"/>
-<instance part="C0897" gate="G$1" x="20.32" y="27.94"/>
-<instance part="C0895" gate="G$1" x="35.56" y="27.94"/>
+<instance part="C0895" gate="G$1" x="20.32" y="27.94"/>
+<instance part="C0897" gate="G$1" x="35.56" y="27.94"/>
 <instance part="L0896" gate="G$1" x="27.94" y="35.56" rot="R270"/>
 <instance part="GND0897" gate="1" x="20.32" y="17.78"/>
@@
 <segment>
 <pinref part="GND0893" gate="1" pin="GND"/>
-<pinref part="C593" gate="G$1" pin="2"/>
+<pinref part="C0891" gate="G$1" pin="2"/>
 <wire x1="20.32" y1="101.6" x2="20.32" y2="104.14" width="0.1524" layer="91"/>
 </segment>
 <segment>
 <pinref part="GND0891" gate="1" pin="GND"/>
-<pinref part="C0891" gate="G$1" pin="2"/>
+<pinref part="C0893" gate="G$1" pin="2"/>
 <wire x1="35.56" y1="101.6" x2="35.56" y2="104.14" width="0.1524" layer="91"/>
 </segment>
@@
 <segment>
 <pinref part="GND0897" gate="1" pin="GND"/>
+<pinref part="C0895" gate="G$1" pin="2"/>
+<wire x1="20.32" y1="20.32" x2="20.32" y2="22.86" width="0.1524" layer="91"/>
+</segment>
+<segment>
+<pinref part="GND0895" gate="1" pin="GND"/>
 <pinref part="C0897" gate="G$1" pin="2"/>
-<wire x1="20.32" y1="20.32" x2="20.32" y2="22.86" width="0.1524" layer="91"/>
-</segment>
-<segment>
-<pinref part="GND0895" gate="1" pin="GND"/>
-<pinref part="C0895" gate="G$1" pin="2"/>
 <wire x1="35.56" y1="20.32" x2="35.56" y2="22.86" width="0.1524" layer="91"/>
 </segment>
@@
 <net name="ANT09" class="7">
 <segment>
-<pinref part="C593" gate="G$1" pin="1"/>
+<pinref part="C0891" gate="G$1" pin="1"/>
 <wire x1="20.32" y1="111.76" x2="20.32" y2="116.84" width="0.1524" layer="91"/>
 <pinref part="L0892" gate="G$1" pin="2"/>
@@
 <net name="ANT09_MATCH" class="7">
 <segment>
-<pinref part="C0891" gate="G$1" pin="1"/>
+<pinref part="C0893" gate="G$1" pin="1"/>
 <wire x1="35.56" y1="111.76" x2="35.56" y2="116.84" width="0.1524" layer="91"/>
 <pinref part="L0892" gate="G$1" pin="1"/>
@@
 <wire x1="15.24" y1="35.56" x2="20.32" y2="35.56" width="0.1524" layer="91"/>
 <pinref part="L0896" gate="G$1" pin="2"/>
-<pinref part="C0897" gate="G$1" pin="1"/>
+<pinref part="C0895" gate="G$1" pin="1"/>
 <wire x1="20.32" y1="35.56" x2="22.86" y2="35.56" width="0.1524" layer="91"/>
 <wire x1="20.32" y1="35.56" x2="20.32" y2="30.48" width="0.1524" layer="91"/>
@@
 <pinref part="L0896" gate="G$1" pin="1"/>
 <wire x1="50.8" y1="35.56" x2="35.56" y2="35.56" width="0.1524" layer="91"/>
-<pinref part="C0895" gate="G$1" pin="1"/>
+<pinref part="C0897" gate="G$1" pin="1"/>
 <wire x1="35.56" y1="35.56" x2="33.02" y2="35.56" width="0.1524" layer="91"/>
 <wire x1="35.56" y1="35.56" x2="35.56" y2="30.48" width="0.1524" layer="91"/>
