File: HW/CAD/Eagle/UFBmod_2V1.brd (EAGLE design)
At the start: 98.4 x 89.5 mm, 204 parts, among them J1411 ABRACON_ARJE-0034, T0551 MMBT2222, U0501 MIDAS_MCCOG21605B6W-FPTLWI, U0601 MAX5217, U0701 AT86RF215-ZU, U0711 ASVTX-13-D-26.000MHZ-I05-T, U0811 PE4259, U0821 RFX1010, U0881 B39871B3440U410, U0911 FT232HL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

Commit message: HW - Eagle - V2.2 - Ethernet magnetics LED resistor values modified (V2.1 also)
Parts:
- R1421, R1422: value 1kR -> 470R
Changed lines of the file:
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@@
 <attribute name="VALUE" x="85.2932" y="49.6824" size="0.8128" layer="28" font="vector" ratio="20" rot="MR270"/>
 </element>
-<element name="R1421" library="df4iah_rcl" package="R0402" value="1kR" x="72.39" y="35.56" smashed="yes" rot="MR90">
+<element name="R1421" library="df4iah_rcl" package="R0402" value="470R" x="72.39" y="35.56" smashed="yes" rot="MR90">
 <attribute name="NAME" x="73.3425" y="34.29" size="0.6096" layer="26" font="vector" ratio="10" rot="MR90"/>
 <attribute name="VALUE" x="70.8025" y="33.9725" size="0.6096" layer="28" font="vector" ratio="10" rot="MR90"/>
 </element>
-<element name="R1422" library="df4iah_rcl" package="R0402" value="1kR" x="72.39" y="53.34" smashed="yes" rot="MR270">
+<element name="R1422" library="df4iah_rcl" package="R0402" value="470R" x="72.39" y="53.34" smashed="yes" rot="MR270">
 <attribute name="NAME" x="72.0725" y="54.9275" size="0.6096" layer="26" font="vector" ratio="10" rot="MR90"/>
 <attribute name="VALUE" x="73.9775" y="54.9275" size="0.6096" layer="28" font="vector" ratio="10" rot="MR270"/>

Commit message: HW - Eagle - V2.1 V2.2 - TRX corrections added
Parts:
- C0703, C0704: value 1nF -> 1uF
- C0713: value 1nF -> N/A
- R0711: value 33R -> 130R
Changed lines of the file:
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@@
 <attribute name="VALUE" x="7.62" y="48.26" size="1.27" layer="27" rot="R270"/>
 </element>
-<element name="C0704" library="df4iah_rcl" package="C0402" value="1nF" x="12.7" y="45.72" smashed="yes" rot="MR180">
+<element name="C0704" library="df4iah_rcl" package="C0402" value="1uF" x="12.7" y="45.72" smashed="yes" rot="MR180">
 <attribute name="NAME" x="13.97" y="46.6725" size="0.6096" layer="26" font="vector" ratio="10" rot="MR0"/>
 <attribute name="VALUE" x="11.43" y="47.3075" size="0.6096" layer="28" font="vector" ratio="10" rot="MR180"/>
 </element>
-<element name="C0703" library="df4iah_rcl" package="C0402" value="1nF" x="19.05" y="32.0675" smashed="yes" rot="MR180">
+<element name="C0703" library="df4iah_rcl" package="C0402" value="1uF" x="19.05" y="32.0675" smashed="yes" rot="MR180">
 <attribute name="NAME" x="21.2725" y="33.02" size="0.6096" layer="26" font="vector" ratio="10" rot="MR0"/>
 <attribute name="VALUE" x="17.78" y="33.655" size="0.6096" layer="28" font="vector" ratio="10" rot="MR180"/>
@@
 <attribute name="VALUE" x="38.4175" y="65.7225" size="0.6096" layer="27" font="vector" ratio="10" rot="R90"/>
 </element>
-<element name="R0711" library="df4iah_rcl" package="R0402" value="33R" x="12.7" y="38.4175" smashed="yes">
+<element name="R0711" library="df4iah_rcl" package="R0402" value="130R" x="12.7" y="38.4175" smashed="yes">
 <attribute name="NAME" x="11.43" y="37.1475" size="0.6096" layer="25" font="vector" ratio="10" rot="R90"/>
 <attribute name="VALUE" x="11.1125" y="36.83" size="0.6096" layer="27" font="vector" ratio="10"/>
@@
 <attribute name="VALUE" x="29.5275" y="50.165" size="0.6096" layer="27" font="vector" ratio="10" rot="R270"/>
 </element>
-<element name="C0713" library="df4iah_rcl" package="C0402" value="1nF" x="12.7" y="36.83" smashed="yes" rot="R180">
+<element name="C0713" library="df4iah_rcl" package="C0402" value="N/A" x="12.7" y="36.83" smashed="yes" rot="R180">
 <attribute name="NAME" x="11.43" y="34.29" size="0.6096" layer="25" font="vector" ratio="10"/>
 <attribute name="VALUE" x="13.97" y="38.4175" size="0.6096" layer="27" font="vector" ratio="10" rot="R180"/>

Commit message: HW - Eagle - V2.1 V2.2 - TRX no 300R inductors at GND lines
Parts:
- L0701, L0702: value 300R -> 0R
Changed lines of the file:
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@@
 <attribute name="VALUE" x="15.17" y="35.89" size="0.6096" layer="27" font="vector" rot="R270" align="top-center"/>
 </element>
-<element name="L0702" library="df4iah_rcl" package="R1206" value="300R" x="20.6375" y="30.1625" smashed="yes" rot="R90">
+<element name="L0702" library="df4iah_rcl" package="R1206" value="0R" x="20.6375" y="30.1625" smashed="yes" rot="R90">
 <attribute name="NAME" x="22.70125" y="28.41625" size="0.6096" layer="25" font="vector" rot="R90"/>
 <attribute name="VALUE" x="23.1775" y="28.8925" size="1.27" layer="27" rot="R90"/>
 </element>
-<element name="L0701" library="df4iah_rcl" package="R1206" value="300R" x="13.97" y="46.99" smashed="yes" rot="R270">
+<element name="L0701" library="df4iah_rcl" package="R1206" value="0R" x="13.97" y="46.99" smashed="yes" rot="R270">
 <attribute name="NAME" x="12.7" y="45.56125" size="0.6096" layer="25" font="vector" rot="R90"/>
 <attribute name="VALUE" x="11.43" y="48.26" size="1.27" layer="27" rot="R270"/>

Commit message: HW - Eagle - V2.1 V2.2 - PMIC values changed for lower swing at VFB and OV-protection
Parts:
- R1103: value 187kR -> N/A
- R1131: value 3.01kR -> 15kR
Changed lines of the file:
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@@
 <attribute name="VALUE" x="78.105" y="80.01" size="0.6096" layer="27" font="vector" ratio="10" rot="R90"/>
 </element>
-<element name="R1103" library="df4iah_rcl" package="R0402" value="187kR" x="67.31" y="85.725" smashed="yes" rot="MR270">
+<element name="R1103" library="df4iah_rcl" package="R0402" value="N/A" x="67.31" y="85.725" smashed="yes" rot="MR270">
 <attribute name="NAME" x="65.7225" y="84.455" size="0.6096" layer="26" font="vector" ratio="10" rot="MR90"/>
 <attribute name="VALUE" x="68.8975" y="87.3125" size="0.6096" layer="28" font="vector" ratio="10" rot="MR270"/>
@@
 <attribute name="VALUE" x="81.28" y="74.295" size="0.6096" layer="27" font="vector" ratio="10"/>
 </element>
-<element name="R1131" library="df4iah_rcl" package="R0402" value="3.01kR" x="74.93" y="69.85" smashed="yes" rot="MR270">
+<element name="R1131" library="df4iah_rcl" package="R0402" value="15kR" x="74.93" y="69.85" smashed="yes" rot="MR270">
 <attribute name="NAME" x="75.8825" y="68.58" size="0.6096" layer="26" font="vector" ratio="10" rot="MR90"/>
 <attribute name="VALUE" x="76.5175" y="71.4375" size="0.6096" layer="28" font="vector" ratio="10" rot="MR270"/>
